File: board/board.kicad_sch (KiCad schematic)
At the start: 1 part

Commit message: initial
Parts:
- removed LOGO1: Logo_Open_Hardware_Small, Symbol:OSHW-Symbol_6.7x6mm_SilkScreen, symbol Graphic:Logo_Open_Hardware_Small
- added J1, J6: (no value), symbol Connector:Conn_01x10_Male
- added J2: CA2310PA10Z, Connector_PinHeader_2.54mm:PinHeader_2x05_P2.54mm_Vertical, symbol Connector:Conn_01x10_Male
Connections:
- new net: J1.1 (Pin_1), J2.1 (Pin_1), J6.1 (Pin_1)
- new net: J1.10 (Pin_10), J2.10 (Pin_10), J6.10 (Pin_10)
- new net: J1.2 (Pin_2), J2.2 (Pin_2), J6.2 (Pin_2)
- new net: J1.3 (Pin_3), J2.3 (Pin_3), J6.3 (Pin_3)
- new net: J1.4 (Pin_4), J2.4 (Pin_4), J6.4 (Pin_4)
- new net: J1.5 (Pin_5), J2.5 (Pin_5), J6.5 (Pin_5)
- new net: J1.6 (Pin_6), J2.6 (Pin_6), J6.6 (Pin_6)
- new net: J1.7 (Pin_7), J2.7 (Pin_7), J6.7 (Pin_7)
- new net: J1.8 (Pin_8), J2.8 (Pin_8), J6.8 (Pin_8)
- new net: J1.9 (Pin_9), J2.9 (Pin_9), J6.9 (Pin_9)
Other:
- removed sheet implementation
- note removed: "Input connectors go here"
- note removed: "Output connectors go here"
Changed lines of the file:
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@@
 (kicad_sch (version 20211123) (generator eeschema)
   (paper "A4")
-  (text "Output connectors go here" (at 224.79 88.9 0)
-    (effects (font (size 1.27 1.27)) (justify left bottom))
+  (junction (at 132.08 105.41) (diameter 0) (color 0 0 0 0)
   )
-  (text "Input connectors go here" (at 49.53 88.9 0)
-    (effects (font (size 1.27 1.27)) (justify left bottom))
+  (junction (at 132.08 90.17) (diameter 0) (color 0 0 0 0)
   )
-  (symbol (lib_id "Graphic:Logo_Open_Hardware_Small") (at 273.05 157.48 0) (unit 1)
-    (in_bom yes) (on_board yes) (fields_autoplaced)
-    (property "Reference" "LOGO1" (id 0) (at 273.05 150.495 0)
+  (junction (at 132.08 95.25) (diameter 0) (color 0 0 0 0)
+  )
+  (junction (at 132.08 102.87) (diameter 0) (color 0 0 0 0)
+  )
+  (junction (at 132.08 97.79) (diameter 0) (color 0 0 0 0)
+  )
+  (junction (at 132.08 100.33) (diameter 0) (color 0 0 0 0)
+  )
+  (junction (at 132.08 92.71) (diameter 0) (color 0 0 0 0)
+  )
+  (junction (at 132.08 87.63) (diameter 0) (color 0 0 0 0)
+  )
+  (junction (at 132.08 82.55) (diameter 0) (color 0 0 0 0)
+  )
+  (junction (at 132.08 85.09) (diameter 0) (color 0 0 0 0)
+  )
+  (wire (pts (xy 124.46 90.17) (xy 132.08 90.17))
+    (stroke (width 0) (type default) (color 0 0 0 0))
+  )
+  (wire (pts (xy 132.08 105.41) (xy 151.13 105.41))
+    (stroke (width 0) (type default) (color 0 0 0 0))
+  )
+  (wire (pts (xy 124.46 85.09) (xy 132.08 85.09))
+    (stroke (width 0) (type default) (color 0 0 0 0))
+  )
+  (wire (pts (xy 124.46 97.79) (xy 132.08 97.79))
+    (stroke (width 0) (type default) (color 0 0 0 0))
+  )
+  (wire (pts (xy 124.46 82.55) (xy 132.08 82.55))
+    (stroke (width 0) (type default) (color 0 0 0 0))
+  )
+  (wire (pts (xy 132.08 87.63) (xy 151.13 87.63))
+    (stroke (width 0) (type default) (color 0 0 0 0))
+  )
+  (wire (pts (xy 132.08 90.17) (xy 151.13 90.17))
+    (stroke (width 0) (type default) (color 0 0 0 0))
+  )
+  (wire (pts (xy 132.08 85.09) (xy 151.13 85.09))
+    (stroke (width 0) (type default) (color 0 0 0 0))
+  )
+  (wire (pts (xy 132.08 102.87) (xy 151.13 102.87))
+    (stroke (width 0) (type default) (color 0 0 0 0))
+  )
+  (wire (pts (xy 124.46 102.87) (xy 132.08 102.87))
+    (stroke (width 0) (type default) (color 0 0 0 0))
+  )
+  (wire (pts (xy 132.08 95.25) (xy 151.13 95.25))
+    (stroke (width 0) (type default) (color 0 0 0 0))
+  )
+  (wire (pts (xy 124.46 105.41) (xy 132.08 105.41))
+    (stroke (width 0) (type default) (color 0 0 0 0))
+  )
+  (wire (pts (xy 124.46 95.25) (xy 132.08 95.25))
+    (stroke (width 0) (type default) (color 0 0 0 0))
+  )
+  (wire (pts (xy 124.46 92.71) (xy 132.08 92.71))
+    (stroke (width 0) (type default) (color 0 0 0 0))
+  )
+  (wire (pts (xy 132.08 82.55) (xy 151.13 82.55))
+    (stroke (width 0) (type default) (color 0 0 0 0))
+  )
+  (wire (pts (xy 132.08 100.33) (xy 151.13 100.33))
+    (stroke (width 0) (type default) (color 0 0 0 0))
+  )
+  (wire (pts (xy 124.46 87.63) (xy 132.08 87.63))
+    (stroke (width 0) (type default) (color 0 0 0 0))
+  )
+  (wire (pts (xy 124.46 100.33) (xy 132.08 100.33))
+    (stroke (width 0) (type default) (color 0 0 0 0))
+  )
+  (wire (pts (xy 132.08 92.71) (xy 151.13 92.71))
+    (stroke (width 0) (type default) (color 0 0 0 0))
+  )
+  (wire (pts (xy 132.08 97.79) (xy 151.13 97.79))
+    (stroke (width 0) (type default) (color 0 0 0 0))
+  )
+  (symbol (lib_id "Connector:Conn_01x10_Male") (at 127 92.71 0) (unit 1)
+    (in_bom yes) (on_board yes)
+    (property "Reference" "J1" (id 0) (at 129.7432 77.9526 0))
+    (property "Value" "" (id 1) (at 129.7432 80.264 0))
+    (property "Footprint" "" (id 2) (at 127 92.71 0)
       (effects (font (size 1.27 1.27)) hide)
     )
-    (property "Value" "Logo_Open_Hardware_Small" (id 1) (at 273.05 163.195 0)
+    (property "Datasheet" "~" (id 3) (at 127 92.71 0)
       (effects (font (size 1.27 1.27)) hide)
     )
-    (property "Footprint" "Symbol:OSHW-Symbol_6.7x6mm_SilkScreen" (id 2) (at 273.05 157.48 0)
+    (pin "1")
+    (pin "10")
+    (pin "2")
+    (pin "3")
+    (pin "4")
+    (pin "5")
+    (pin "6")
+    (pin "7")
+    (pin "8")
+    (pin "9")
+  )
+  (symbol (lib_id "Connector:Conn_01x10_Male") (at 119.38 92.71 0) (unit 1)
+    (in_bom yes) (on_board yes)
+    (property "Reference" "J6" (id 0) (at 122.1232 77.9526 0))
+    (property "Value" "" (id 1) (at 122.1232 80.264 0))
+    (property "Footprint" "" (id 2) (at 119.38 92.71 0)
       (effects (font (size 1.27 1.27)) hide)
     )
-    (property "Datasheet" "~" (id 3) (at 273.05 157.48 0)
+    (property "Datasheet" "~" (id 3) (at 119.38 92.71 0)
       (effects (font (size 1.27 1.27)) hide)
     )
+    (pin "1")
+    (pin "10")
+    (pin "2")
+    (pin "3")
+    (pin "4")
+    (pin "5")
+    (pin "6")
+    (pin "7")
+    (pin "8")
+    (pin "9")
   )
-  (sheet (at 114.3 72.39) (size 60.96 62.23) (fields_autoplaced)
-    (stroke (width 0.1524) (type solid) (color 0 0 0 0))
-    (fill (color 0 0 0 0.0000))
-    (property "Sheet name" "implementation" (id 0) (at 114.3 71.6784 0)
-      (effects (font (size 1.27 1.27)) (justify left bottom))
+  (symbol (lib_id "Connector:Conn_01x10_Male") (at 146.05 92.71 0) (unit 1)
+    (in_bom yes) (on_board yes)
+    (property "Reference" "J2" (id 0) (at 148.7932 77.9526 0))
+    (property "Value" "CA2310PA10Z" (id 1) (at 148.7932 80.264 0))
+    (property "Footprint" "Connector_PinHeader_2.54mm:PinHeader_2x05_P2.54mm_Vertical" (id 2) (at 146.05 92.71 0)
+      (effects (font (size 1.27 1.27)) hide)
     )
-    (property "Sheet file" "implementation.kicad_sch" (id 1) (at 114.3 135.2046 0)
-      (effects (font (size 1.27 1.27)) (justify left top))
+    (property "Datasheet" "~" (id 3) (at 146.05 92.71 0)
+      (effects (font (size 1.27 1.27)) hide)
     )
+    (pin "1")
+    (pin "10")
+    (pin "2")
+    (pin "3")
+    (pin "4")
+    (pin "5")
+    (pin "6")
+    (pin "7")
+    (pin "8")
+    (pin "9")
   )
   (sheet_instances
     (path "/" (page "1"))
-    (path "/767ce4c6-0e55-4543-92f0-34cb8237a544" (page "2"))
   )
   (symbol_instances
-    (path "/b72b6f4a-7489-40f2-bb90-d75ae01aa368"
-      (reference "LOGO1") (unit 1) (value "Logo_Open_Hardware_Small") (footprint "Symbol:OSHW-Symbol_6.7x6mm_SilkScreen")
+    (path "/00000000-0000-0000-0000-0000602487d2"
+      (reference "J1") (unit 1) (value "Conn_01x10_Male") (footprint "on_edge:on_edge_2x05_device")
+    )
+    (path "/3e425ab4-13b7-4cfe-9de4-bcc68d4f7f06"
+      (reference "J2") (unit 1) (value "CA2310PA10Z") (footprint "Connector_PinHeader_2.54mm:PinHeader_2x05_P2.54mm_Vertical")
+    )
+    (path "/00000000-0000-0000-0000-0000602592e9"
+      (reference "J6") (unit 1) (value "Conn_01x10_Male") (footprint "on_edge:on_edge_2x05_host")
     )
   )
